Commit message: Operated Bot with Keyboard and RVz2 and gazebo launch in a single command and synced

File: description/robot.urdf.xacro (robot description, xacro)
@@ -2,3 +2,4 @@
 <robot xmlns:xacro="http://www.ros.org/wiki/xacro"  name="robot">
   <xacro:include filename="robot_core.xacro" />
+  <xacro:include filename="gazebo_control.xacro" />
 </robot>

File: description/robot_core.xacro (robot description, xacro)
@@ -2,16 +2,22 @@
 <robot xmlns:xacro="http://www.ros.org/wiki/xacro" >
     <xacro:include filename="inertial_macros.xacro" />
-    <!-- ==================== MATERIALS ==================== -->
+    <!-- ==================== MATERIALS (RViz colors) ==================== -->
     <material name="white">
         <color rgba="1 1 1 1"/>
     </material>
     <material name="orange">
-        <color rgba="1 0.5 0 1"/>
+        <color rgba="1 0.3 0 1"/>
     </material>
     <material name="blue">
-        <color rgba="0 0 1 1"/>
+        <color rgba="0.1 0.1 0.8 1"/>
     </material>
     <material name="black">
-        <color rgba="0 0 0 1"/>
+        <color rgba="0.05 0.05 0.05 1"/>
+    </material>
+    <material name="dark_grey">
+        <color rgba="0.2 0.2 0.2 1"/>
+    </material>
+    <material name="silver">
+        <color rgba="0.75 0.75 0.75 1"/>
     </material>
     <!-- Base Link -->
@@ -30,5 +36,5 @@
                 <box size="0.3 0.3 0.15"/>
             </geometry>
-            <material name="white"/>
+            <material name="orange"/>
         </visual>
         <collision>
@@ -55,5 +61,5 @@
                 <cylinder radius="0.05" length="0.04"/>
             </geometry>
-            <material name="blue"/>
+            <material name="dark_grey"/>
         </visual>
         <collision>
@@ -80,5 +86,5 @@
                 <cylinder radius="0.05" length="0.04"/>
             </geometry>
-            <material name="blue"/>
+            <material name="dark_grey"/>
         </visual>
         <collision>
@@ -103,5 +109,5 @@
                 <sphere radius="0.05"/>
             </geometry>
-            <material name="black"/>
+            <material name="silver"/>
         </visual>
         <collision>
@@ -114,3 +120,38 @@
         </xacro:inertial_sphere>
     </link>
-    </robot>
+    <!-- ==================== GAZEBO COLORS ==================== -->
+    <!-- Gazebo Harmonic uses these tags to apply colors in simulation -->
+    <!-- Chassis: Orange -->
+    <gazebo reference="chassis">
+        <material>
+            <ambient>1.0 0.3 0.0 1</ambient>
+            <diffuse>1.0 0.3 0.0 1</diffuse>
+            <specular>0.6 0.6 0.6 1</specular>
+        </material>
+    </gazebo>
+    <!-- Wheels: Dark Grey -->
+    <gazebo reference="left_wheel">
+        <material>
+            <ambient>0.2 0.2 0.2 1</ambient>
+            <diffuse>0.2 0.2 0.2 1</diffuse>
+            <specular>0.3 0.3 0.3 1</specular>
+        </material>
+    </gazebo>
+    <gazebo reference="right_wheel">
+        <material>
+            <ambient>0.2 0.2 0.2 1</ambient>
+            <diffuse>0.2 0.2 0.2 1</diffuse>
+            <specular>0.3 0.3 0.3 1</specular>
+        </material>
+    </gazebo>
+    <!-- Caster: Silver with low friction -->
+    <gazebo reference="caster_wheel">
+        <mu1 value="0.001"/>
+        <mu2 value="0.001"/>
+        <material>
+            <ambient>0.75 0.75 0.75 1</ambient>
+            <diffuse>0.75 0.75 0.75 1</diffuse>
+            <specular>0.8 0.8 0.8 1</specular>
+        </material>
+    </gazebo>
+</robot>

Commit message: Lidar added as well as  launch script for physical lidar testing

File: description/robot.urdf.xacro (robot description, xacro)
@@ -3,3 +3,4 @@
   <xacro:include filename="robot_core.xacro" />
   <xacro:include filename="gazebo_control.xacro" />
+  <xacro:include filename="lidar.xacro" />
 </robot>

File: description/robot_core.xacro (robot description, xacro)
@@ -20,4 +20,7 @@
     <material name="silver">
         <color rgba="0.75 0.75 0.75 1"/>
+    </material>
+    <material name="red">
+        <color rgba="1 0 0 1"/>
     </material>
     <!-- Base Link -->
@@ -147,6 +150,6 @@
     <!-- Caster: Silver with low friction -->
     <gazebo reference="caster_wheel">
-        <mu1 value="0.001"/>
-        <mu2 value="0.001"/>
+        <mu1>0.001</mu1>
+        <mu2>0.001</mu2>
         <material>
             <ambient>0.75 0.75 0.75 1</ambient>
