Commit message: Done with slam tool box and map generation

File: description/camera.xacro (robot description, xacro)
@@ -6,5 +6,5 @@
         <parent link="chassis"/>
         <child link="camera_link"/>
-        <origin xyz="0.27 0 0.15" rpy="0 0 0"/>
+        <origin xyz="0.305 0 0.08" rpy="0 0 0"/>
     </joint>
     <!-- Camera link (small box representing the camera body) -->

File: description/robot.urdf.xacro (robot description, xacro)
@@ -2,6 +2,7 @@
 <robot xmlns:xacro="http://www.ros.org/wiki/xacro"  name="robot">
   <xacro:include filename="robot_core.xacro" />
-  <xacro:include filename="gazebo_control.xacro" />
   <xacro:include filename="lidar.xacro" />
   <xacro:include filename="camera.xacro" />
+  <!--<xacro:include filename="gazebo_control.xacro" />-->
+  <xacro:include filename="ros2_control.xacro" />
 </robot>

File: description/robot_core.xacro (robot description, xacro)
@@ -27,4 +27,11 @@
     <link name="base_link">
     </link>
+    <!--   Base FOOTPRINT LINK  -->
+    <joint name="base_footprint_joint" type="fixed">
+        <parent link="base_link"/>
+        <child link="base_footprint"/>
+        <origin xyz="0 0 0" rpy="0 0 0"/>
+    </joint>
+    <link name="base_footprint"> </link>
     <!-- Chasis LINK -->
     <joint name="chasis_joint" type="fixed">
@@ -47,5 +54,5 @@
             </geometry>
         </collision>
-        <xacro:inertial_box mass="0.5" x="0.3" y="0.3" z="0.15">
+        <xacro:inertial_box mass="1.5" x="0.3" y="0.3" z="0.15">
             <origin xyz="0.15 0 0.075" rpy="0 0 0"/>
         </xacro:inertial_box>
@@ -69,5 +76,5 @@
             <origin xyz="0 0 0" rpy="0 0 0"/>
             <geometry>
-                <cylinder radius="0.05" length="0.04"/>
+                <sphere radius="0.05"/>
             </geometry>
         </collision>
@@ -94,5 +101,5 @@
             <origin xyz="0 0 0" rpy="0 0 0"/>
             <geometry>
-                <cylinder radius="0.05" length="0.04"/>
+                <sphere radius="0.05"/>
             </geometry>
         </collision>
@@ -133,6 +140,12 @@
         </material>
     </gazebo>
-    <!-- Wheels: Dark Grey -->
+    <!-- Wheels: Dark Grey with high friction for traction -->
     <gazebo reference="left_wheel">
+        <mu1>100</mu1>
+        <mu2>50</mu2>
+        <kp>1000000.0</kp>
+        <kd>1.0</kd>
+        <minDepth>0.001</minDepth>
+        <maxVel>0.0</maxVel>
         <material>
             <ambient>0.2 0.2 0.2 1</ambient>
@@ -142,4 +155,10 @@
     </gazebo>
     <gazebo reference="right_wheel">
+        <mu1>100</mu1>
+        <mu2>50</mu2>
+        <kp>1000000.0</kp>
+        <kd>1.0</kd>
+        <minDepth>0.001</minDepth>
+        <maxVel>0.0</maxVel>
         <material>
             <ambient>0.2 0.2 0.2 1</ambient>
@@ -148,8 +167,12 @@
         </material>
     </gazebo>
-    <!-- Caster: Silver with low friction -->
+    <!-- Caster: Silver with near-zero friction for free pivot -->
     <gazebo reference="caster_wheel">
         <mu1>0.001</mu1>
         <mu2>0.001</mu2>
+        <kp>1000000.0</kp>
+        <kd>1.0</kd>
+        <minDepth>0.001</minDepth>
+        <maxVel>0.0</maxVel>
         <material>
             <ambient>0.75 0.75 0.75 1</ambient>
