Commit message: feat: update for JGB37-520 DC12V 110RPM motors with 65mm wheels
Motor: JGB37-520 with Hall encoder (11 PPR, ~90:1 gear ratio)
- ticks_per_rev: 1320 -> 990 (11 PPR x 90:1 gear)
- wheel_radius: 0.05m -> 0.0325m (65mm diameter wheels)
- wheel_width: 0.04m -> 0.026m (65x26mm wheels)
- max_motor_speed: 0.5 -> 0.37 m/s (110RPM x pi x 0.065m)

Updated files:
- firmware/motor_controller.ino: JGB37-520 6-pin connector wiring docs
- scripts/diff_drive_node.py: motor params and docstring
- launch/bringup_hardware.launch.py: default parameters
- description/robot_core.xacro: wheel/caster dimensions
- COMPLETE_GUIDE.md: wiring guide for JGB37-520 6-pin connector
- HARDWARE_DEPLOYMENT.md: motor and wheel specs

File: description/robot_core.xacro (robot description, xacro)
@@ -69,5 +69,5 @@
             <origin xyz="0 0 0" rpy="0 0 0"/>
             <geometry>
-                <cylinder radius="0.05" length="0.04"/>
+                <cylinder radius="0.0325" length="0.026"/>
             </geometry>
             <material name="dark_grey"/>
@@ -76,8 +76,8 @@
             <origin xyz="0 0 0" rpy="0 0 0"/>
             <geometry>
-                <sphere radius="0.05"/>
+                <sphere radius="0.0325"/>
             </geometry>
         </collision>
-        <xacro:inertial_cylinder mass="0.1" length="0.04" radius="0.05">
+        <xacro:inertial_cylinder mass="0.1" length="0.026" radius="0.0325">
             <origin xyz="0 0 0" rpy="0 0 0"/>
         </xacro:inertial_cylinder>
@@ -94,5 +94,5 @@
             <origin xyz="0 0 0" rpy="0 0 0"/>
             <geometry>
-                <cylinder radius="0.05" length="0.04"/>
+                <cylinder radius="0.0325" length="0.026"/>
             </geometry>
             <material name="dark_grey"/>
@@ -101,8 +101,8 @@
             <origin xyz="0 0 0" rpy="0 0 0"/>
             <geometry>
-                <sphere radius="0.05"/>
+                <sphere radius="0.0325"/>
             </geometry>
         </collision>
-        <xacro:inertial_cylinder mass="0.1" length="0.04" radius="0.05">
+        <xacro:inertial_cylinder mass="0.1" length="0.026" radius="0.0325">
             <origin xyz="0 0 0" rpy="0 0 0"/>
         </xacro:inertial_cylinder>
@@ -117,5 +117,5 @@
         <visual>
             <geometry>
-                <sphere radius="0.05"/>
+                <sphere radius="0.0325"/>
             </geometry>
             <material name="silver"/>
@@ -123,8 +123,8 @@
         <collision>
             <geometry>
-                <sphere radius="0.05"/>
+                <sphere radius="0.0325"/>
             </geometry>
         </collision>
-        <xacro:inertial_sphere mass="0.1" radius="0.05">
+        <xacro:inertial_sphere mass="0.1" radius="0.0325">
             <origin xyz="0 0 0" rpy="0 0 0"/>
         </xacro:inertial_sphere>
