Commit message: fix: add motor housings, caster mount bracket, and LiDAR riser post
- Add left/right motor cylinders (r=14mm, l=40mm) between support posts
  and wheels, giving the drive system a visible motor body
- Add caster mount bracket (20x15x40mm silver box) connecting the chassis
  bottom to the caster ball, eliminating the floating gap
- Add LiDAR riser post (40x40x25mm wood block) between chassis top and
  LiDAR bottom, so the sensor sits on a visible support
- Add Gazebo material colors for all new links

File: description/gazebo_control.xacro (robot description, xacro)
@@ -63,4 +63,28 @@
     </material>
   </gazebo>
+  <gazebo reference="left_motor">
+    <material>
+      <ambient>0.2 0.2 0.2 1</ambient>
+      <diffuse>0.2 0.2 0.2 1</diffuse>
+    </material>
+  </gazebo>
+  <gazebo reference="right_motor">
+    <material>
+      <ambient>0.2 0.2 0.2 1</ambient>
+      <diffuse>0.2 0.2 0.2 1</diffuse>
+    </material>
+  </gazebo>
+  <gazebo reference="caster_mount">
+    <material>
+      <ambient>0.75 0.75 0.75 1</ambient>
+      <diffuse>0.75 0.75 0.75 1</diffuse>
+    </material>
+  </gazebo>
+  <gazebo reference="lidar_riser">
+    <material>
+      <ambient>0.76 0.60 0.42 1</ambient>
+      <diffuse>0.76 0.60 0.42 1</diffuse>
+    </material>
+  </gazebo>
   <!-- Caster wheel: low friction for free rolling -->
   <gazebo reference="caster_wheel">

File: description/robot_core.xacro (robot description, xacro)
@@ -120,4 +120,41 @@
         </visual>
     </link>
+    <!-- ==================== MOTOR HOUSINGS ==================== -->
+    <!--
+      DC motor cylinders between support posts and wheels.
+      Oriented along Y axis (perpendicular to chassis).
+      Radius ~14mm, length ~40mm — bridges from support post to wheel.
+      Centered at wheel X position, between post and wheel in Y.
+    -->
+    <!-- Left motor -->
+    <joint name="left_motor_joint" type="fixed">
+        <parent link="chassis"/>
+        <child link="left_motor"/>
+        <origin xyz="0.147 0.065 0" rpy="0 0 0"/>
+    </joint>
+    <link name="left_motor">
+        <visual>
+            <origin xyz="0 0 0" rpy="${pi/2} 0 0"/>
+            <geometry>
+                <cylinder radius="0.014" length="0.040"/>
+            </geometry>
+            <material name="dark_grey"/>
+        </visual>
+    </link>
+    <!-- Right motor -->
+    <joint name="right_motor_joint" type="fixed">
+        <parent link="chassis"/>
+        <child link="right_motor"/>
+        <origin xyz="0.147 -0.065 0" rpy="0 0 0"/>
+    </joint>
+    <link name="right_motor">
+        <visual>
+            <origin xyz="0 0 0" rpy="${pi/2} 0 0"/>
+            <geometry>
+                <cylinder radius="0.014" length="0.040"/>
+            </geometry>
+            <material name="dark_grey"/>
+        </visual>
+    </link>
     <!-- ==================== LEFT WHEEL ==================== -->
     <!--
@@ -175,4 +212,24 @@
         </xacro:inertial_cylinder>
     </link>
+    <!-- ==================== CASTER MOUNT BRACKET ==================== -->
+    <!--
+      Vertical bracket connecting chassis bottom (z=0.035) to caster area.
+      Fills the visual gap between the chassis plate and the caster ball.
+      Height: 40mm, from z=-0.005 to z=0.035 (chassis bottom).
+    -->
+    <joint name="caster_mount_joint" type="fixed">
+        <parent link="chassis"/>
+        <child link="caster_mount"/>
+        <origin xyz="0.337 0 0.015" rpy="0 0 0"/>
+    </joint>
+    <link name="caster_mount">
+        <visual>
+            <origin xyz="0 0 0" rpy="0 0 0"/>
+            <geometry>
+                <box size="0.020 0.015 0.040"/>
+            </geometry>
+            <material name="silver"/>
+        </visual>
+    </link>
     <!-- ==================== CASTER WHEEL ==================== -->
     <!--
@@ -202,3 +259,23 @@
         </xacro:inertial_sphere>
     </link>
+    <!-- ==================== LIDAR RISER POST ==================== -->
+    <!--
+      Wooden post supporting the LiDAR above the chassis.
+      Fills the gap between chassis top (z=0.055) and LiDAR bottom (z=0.08).
+      Height: 25mm, centered at z=0.0675, at LiDAR x position.
+    -->
+    <joint name="lidar_riser_joint" type="fixed">
+        <parent link="chassis"/>
+        <child link="lidar_riser"/>
+        <origin xyz="0.106 0 0.0675" rpy="0 0 0"/>
+    </joint>
+    <link name="lidar_riser">
+        <visual>
+            <origin xyz="0 0 0" rpy="0 0 0"/>
+            <geometry>
+                <box size="0.040 0.040 0.025"/>
+            </geometry>
+            <material name="wood"/>
+        </visual>
+    </link>
 </robot>

Commit message: fix: move LiDAR to rear edge, replace gz_ros2_control with DiffDrive plugin
Issues fixed:
1. LiDAR moved from x=0.106 to x=0.04 (near chassis rear edge)
   Both lidar_sim.xacro and robot_core.xacro (riser post) updated

2. Robot not moving: replaced gz_ros2_control + ros2_controllers with
   Gazebo's built-in DiffDrive system plugin. Teleop now works with
   just 'ros2 run teleop_twist_keyboard teleop_twist_keyboard'
   (no --ros-args remapping needed)

3. SLAM not receiving scan data: changed sensor topic from relative
   'scan' to absolute '/scan' so ros_gz_bridge finds it correctly.
   Added full bridge for /cmd_vel, /odom, /tf, /joint_states, /scan, /clock

Removed gz_ros2_control dependency and controller spawners from launch.

File: description/gazebo_control.xacro (robot description, xacro)
@@ -2,32 +2,37 @@
 <robot xmlns:xacro="http://www.ros.org/wiki/xacro">
   <!--
-    Gazebo Harmonic (gz-sim) ros2_control integration
-    Uses gz_ros2_control plugin to drive the DiffDriveController
-    defined in my_controllers.yaml through Gazebo simulation.
+    Gazebo Harmonic (gz-sim) — Differential Drive + Joint State Publisher
+    Uses Gazebo's built-in DiffDrive system plugin for motor control.
+    Teleop_twist_keyboard publishes to /cmd_vel and the robot moves directly.
+    No ros2_control needed — simpler and more reliable for simulation.
   -->
-  <ros2_control name="GazeboSimSystem" type="system">
-    <hardware>
-      <plugin>gz_ros2_control/GazeboSimSystem</plugin>
-    </hardware>
-    <joint name="left_wheel_joint">
-      <command_interface name="velocity">
-        <param name="min">-10</param>
-        <param name="max">10</param>
-      </command_interface>
-      <state_interface name="position"/>
-      <state_interface name="velocity"/>
-    </joint>
-    <joint name="right_wheel_joint">
-      <command_interface name="velocity">
-        <param name="min">-10</param>
-        <param name="max">10</param>
-      </command_interface>
-      <state_interface name="position"/>
-      <state_interface name="velocity"/>
-    </joint>
-  </ros2_control>
+  <!-- ==================== DIFFERENTIAL DRIVE PLUGIN ==================== -->
   <gazebo>
-    <plugin filename="gz_ros2_control-system" name="gz_ros2_control::GazeboSimROS2ControlPlugin">
-      <parameters>$(find my_bot)/config/my_controllers.yaml</parameters>
+    <plugin filename="gz-sim-diff-drive-system" name="gz::sim::systems::DiffDrive">
+      <left_joint>left_wheel_joint</left_joint>
+      <right_joint>right_wheel_joint</right_joint>
+      <wheel_separation>0.181</wheel_separation>
+      <wheel_radius>0.0345</wheel_radius>
+      <max_linear_acceleration>1.0</max_linear_acceleration>
+      <min_linear_acceleration>-1.0</min_linear_acceleration>
+      <max_angular_acceleration>3.0</max_angular_acceleration>
+      <min_angular_acceleration>-3.0</min_angular_acceleration>
+      <max_linear_velocity>0.47</max_linear_velocity>
+      <max_angular_velocity>2.5</max_angular_velocity>
+      <odom_publish_frequency>30</odom_publish_frequency>
+      <topic>/cmd_vel</topic>
+      <odom_topic>/odom</odom_topic>
+      <tf_topic>/tf</tf_topic>
+      <frame_id>odom</frame_id>
+      <child_frame_id>base_link</child_frame_id>
+    </plugin>
+  </gazebo>
+  <!-- ==================== JOINT STATE PUBLISHER ==================== -->
+  <gazebo>
+    <plugin filename="gz-sim-joint-state-publisher-system" name="gz::sim::systems::JointStatePublisher">
+      <joint_name>left_wheel_joint</joint_name>
+      <joint_name>right_wheel_joint</joint_name>
+      <topic>/joint_states</topic>
+      <update_rate>30</update_rate>
     </plugin>
   </gazebo>

File: description/lidar_sim.xacro (robot description, xacro)
@@ -3,14 +3,14 @@
   <!--
     RPLidar C1 — Simulation Version (Gazebo Harmonic GPU LiDAR)
-    Physical placement identical to hardware:
-      - 106 mm from rear edge of chassis (toward front)
+    Physical placement:
+      - Near the rear edge of the chassis (x=0.04 in chassis frame)
       - Centered laterally (y = 0)
-      - Mounted on top of chassis, ~0.10m above base_link
-      - Relative to chassis link origin (at rear edge): x=0.106, y=0, z=0.10
+      - Mounted on a wooden riser above the chassis, ~0.10m above base_link
+      - Relative to chassis link origin (at rear edge): x=0.04, y=0, z=0.10
     Simulated using Gazebo gpu_lidar sensor, bridged to ROS /scan via ros_gz_bridge.
     RPLidar C1 specifications:
       - Range: 0.15 m to 8.0 m
       - 360° scan
-      - ~4000 samples per revolution
+      - 720 samples per revolution
       - Scan rate: ~10 Hz
   -->
@@ -18,5 +18,5 @@
     <parent link="chassis"/>
     <child link="laser_frame"/>
-    <origin xyz="0.106 0 0.10" rpy="0 0 0"/>
+    <origin xyz="0.04 0 0.10" rpy="0 0 0"/>
   </joint>
   <link name="laser_frame">
@@ -44,5 +44,5 @@
     </material>
     <sensor name="gpu_lidar" type="gpu_lidar">
-      <topic>scan</topic>
+      <topic>/scan</topic>
       <update_rate>10</update_rate>
       <gz_frame_id>laser_frame</gz_frame_id>

File: description/robot_core.xacro (robot description, xacro)
@@ -263,10 +263,11 @@
       Wooden post supporting the LiDAR above the chassis.
       Fills the gap between chassis top (z=0.055) and LiDAR bottom (z=0.08).
-      Height: 25mm, centered at z=0.0675, at LiDAR x position.
+      Height: 25mm, centered at z=0.0675.
+      Placed near the rear edge of the chassis (x=0.04 in chassis frame).
     -->
     <joint name="lidar_riser_joint" type="fixed">
         <parent link="chassis"/>
         <child link="lidar_riser"/>
-        <origin xyz="0.106 0 0.0675" rpy="0 0 0"/>
+        <origin xyz="0.04 0 0.0675" rpy="0 0 0"/>
     </joint>
     <link name="lidar_riser">
