Commit message: feat: migrate to LattePanda Alpha + Arduino Leonardo for Daniel's robot
Hardware changes:
- LattePanda Alpha (Core i5) replaces Orange Pi 5
- Built-in Arduino Leonardo replaces Arduino Uno
- 130 RPM 12V DC motors with 11 PPR quadrature encoders
- L298N H-Bridge motor driver with updated pin mapping
- RPLidar C1 via USB

URDF updates:
- Chassis: 437×212×20mm wood platform on supports
- Wheels: 69mm diameter, 26mm width, 181mm center-to-center
- Caster: 15mm radius front passive wheel at 190mm from drive axle
- LiDAR: 106mm from rear edge, centered, ~100mm above base_link
- Total robot mass: 2.4 kg with proper inertia matrices
- base_footprint at ground plane (z = -0.0345 from base_link)

Arduino Leonardo firmware:
- Updated pin assignments (ENA→D5, IN1→D7, IN2→D6, IN3→D10, IN4→D9, ENB→D11)
- Left encoder: D3 (INT0) + D2 (direction) - hardware interrupt
- Right encoder: A4 + A5 - polling (no HW interrupt on ATmega32U4)
- PID speed control with per-motor feedforward calibration
- USB CDC serial (native USB on Leonardo)

Config updates:
- Nav2 params tuned for LattePanda i5 (higher frequencies)
- SLAM Toolbox optimized for more compute power
- Robot radius updated (0.15m)
- Conservative velocities for 130 RPM motors
- udev rules for Arduino Leonardo (vendor 2341, product 8036/0036)

Cleanup:
- Removed all Gazebo simulation files
- Removed Orange Pi 5 specific scripts
- Removed unused launch files and configs
- Removed worlds directory
- Removed camera, sim ros2_control, and Gazebo plugins

Documentation:
- INSTALLATION_GUIDE.md: Full Ubuntu + ROS2 + hardware setup
- RUNNING_GUIDE.md: Bringup, SLAM, Nav2, troubleshooting
- README.md: Updated project overview and specs

File: description/lidar_hardware.xacro (robot description, xacro)
@@ -2,17 +2,22 @@
 <robot xmlns:xacro="http://www.ros.org/wiki/xacro">
   <!--
-    Lidar link/joint for real hardware.
-    Same physical placement as simulation, but NO Gazebo sensor plugin.
-    The real RPLidar C1 publishes /scan via rplidar_ros driver.
+    RPLidar C1 — Real Hardware Link/Joint
+    Physical placement on Daniel's robot:
+      - 106 mm from rear edge of chassis (toward front)
+      - Centered laterally (y = 0)
+      - Mounted on top of chassis, ~0.10m above base_link
+      - Relative to chassis link origin (at rear edge): x=0.106, y=0, z=0.10
+    The real RPLidar C1 publishes /scan via rplidar_ros driver node.
+    No Gazebo sensor plugin needed.
   -->
   <joint name="laser_joint" type="fixed">
     <parent link="chassis"/>
     <child link="laser_frame"/>
-    <origin xyz="0.1 0 0.175" rpy="0 0 0"/>
+    <origin xyz="0.106 0 0.10" rpy="0 0 0"/>
   </joint>
   <link name="laser_frame">
     <visual>
       <geometry>
-        <cylinder length="0.04" radius="0.05"/>
+        <cylinder length="0.04" radius="0.035"/>
       </geometry>
       <material name="red">
@@ -22,11 +27,11 @@
     <collision>
       <geometry>
-        <cylinder length="0.04" radius="0.05"/>
+        <cylinder length="0.04" radius="0.035"/>
       </geometry>
     </collision>
-    <xacro:inertial_cylinder mass="0.1" length="0.04" radius="0.05">
+    <xacro:inertial_cylinder mass="0.15" length="0.04" radius="0.035">
       <origin xyz="0 0 0" rpy="0 0 0"/>
     </xacro:inertial_cylinder>
   </link>
-  <!-- No Gazebo sensor plugin — real RPLidar provides /scan topic -->
+  <!-- No Gazebo sensor plugin — real RPLidar C1 provides /scan topic -->
 </robot>

File: description/robot_core.xacro (robot description, xacro)
@@ -2,4 +2,25 @@
 <robot xmlns:xacro="http://www.ros.org/wiki/xacro" >
     <xacro:include filename="inertial_macros.xacro" />
+    <!-- ==================== ROBOT PARAMETERS ==================== -->
+    <!--
+      Daniel's Robot — LattePanda Alpha + Arduino Leonardo
+      Differential drive: 2 rear powered wheels + 1 front caster
+      Physical dimensions (from measurements):
+        Length:  0.437 m
+        Width:   0.212 m
+        Height:  0.089 m (ground to chassis top, excl. lidar/computer)
+        Weight:  2.4 kg total
+      Wheels:
+        Diameter: 69 mm  (radius 0.0345 m)
+        Width:    26 mm  (0.026 m)
+        Outer-edge separation: 207 mm
+        Center-to-center:      181 mm  (0.181 m)
+      Drive axle: 147 mm from rear edge
+      Caster:     190 mm forward of drive axle
+      LiDAR:      106 mm from rear edge, centered laterally
+      Coordinate convention:
+        base_link at drive axle center, X-forward, Z-up
+        base_footprint at ground plane (z = -wheel_radius)
+    -->
     <!-- ==================== MATERIALS (RViz colors) ==================== -->
     <material name="white">
@@ -24,43 +45,89 @@
         <color rgba="1 0 0 1"/>
     </material>
-    <!-- Base Link -->
-    <link name="base_link">
-    </link>
-    <!--   Base FOOTPRINT LINK  -->
+    <material name="wood">
+        <color rgba="0.76 0.60 0.42 1"/>
+    </material>
+    <!-- ==================== BASE LINK ==================== -->
+    <link name="base_link"> </link>
+    <!-- ==================== BASE FOOTPRINT (ground plane) ==================== -->
     <joint name="base_footprint_joint" type="fixed">
         <parent link="base_link"/>
         <child link="base_footprint"/>
-        <origin xyz="0 0 0" rpy="0 0 0"/>
+        <origin xyz="0 0 -0.0345" rpy="0 0 0"/>
     </joint>
     <link name="base_footprint"> </link>
-    <!-- Chasis LINK -->
-    <joint name="chasis_joint" type="fixed">
+    <!-- ==================== CHASSIS ==================== -->
+    <!--
+      Chassis = wooden platform (0.437 x 0.212 x 0.020 m)
+      Mounted on vertical supports above the wheels.
+      Bottom of chassis at z=0.035 (just above wheel tops at 0.0345)
+      Top of chassis at z=0.055 above base_link
+      Total height from ground: 0.0345 + 0.055 = 0.0895 m ≈ 89 mm ✓
+    -->
+    <joint name="chassis_joint" type="fixed">
         <parent link="base_link"/>
         <child link="chassis"/>
-        <origin xyz="-0.1 0 0" rpy="0 0 0"/>
+        <origin xyz="-0.147 0 0" rpy="0 0 0"/>
     </joint>
     <link name="chassis">
         <visual>
-            <origin xyz="0.15 0 0.075" rpy="0 0 0"/>
-            <geometry>
-                <box size="0.3 0.3 0.15"/>
-            </geometry>
-            <material name="orange"/>
-        </visual>
-        <collision>
-            <origin xyz="0.15 0 0.075" rpy="0 0 0"/>
-            <geometry>
-                <box size="0.3 0.3 0.15"/>
-            </geometry>
-        </collision>
-        <xacro:inertial_box mass="1.5" x="0.3" y="0.3" z="0.15">
-            <origin xyz="0.15 0 0.075" rpy="0 0 0"/>
+            <origin xyz="0.2185 0 0.045" rpy="0 0 0"/>
+            <geometry>
+                <box size="0.437 0.212 0.020"/>
+            </geometry>
+            <material name="wood"/>
+        </visual>
+        <collision>
+            <origin xyz="0.2185 0 0.045" rpy="0 0 0"/>
+            <geometry>
+                <box size="0.437 0.212 0.020"/>
+            </geometry>
+        </collision>
+        <xacro:inertial_box mass="2.0" x="0.437" y="0.212" z="0.020">
+            <origin xyz="0.2185 0 0.045" rpy="0 0 0"/>
         </xacro:inertial_box>
     </link>
-    <!-- LEFT WHEEL LINK -->
+    <!-- ==================== WHEEL SUPPORT POSTS ==================== -->
+    <!-- Vertical wood support connecting chassis to motor/axle mount area -->
+    <!-- Left support post -->
+    <joint name="left_support_joint" type="fixed">
+        <parent link="chassis"/>
+        <child link="left_support"/>
+        <origin xyz="0.147 0.07 0" rpy="0 0 0"/>
+    </joint>
+    <link name="left_support">
+        <visual>
+            <origin xyz="0 0 0.0175" rpy="0 0 0"/>
+            <geometry>
+                <box size="0.04 0.02 0.035"/>
+            </geometry>
+            <material name="wood"/>
+        </visual>
+    </link>
+    <!-- Right support post -->
+    <joint name="right_support_joint" type="fixed">
+        <parent link="chassis"/>
+        <child link="right_support"/>
+        <origin xyz="0.147 -0.07 0" rpy="0 0 0"/>
+    </joint>
+    <link name="right_support">
+        <visual>
+            <origin xyz="0 0 0.0175" rpy="0 0 0"/>
+            <geometry>
+                <box size="0.04 0.02 0.035"/>
+            </geometry>
+            <material name="wood"/>
+        </visual>
+    </link>
+    <!-- ==================== LEFT WHEEL ==================== -->
+    <!--
+      Center-to-center wheel separation: 0.181 m
+      Each wheel at y = ±0.0905 m from base_link
+      Wheel: radius 0.0345m, width 0.026m
+    -->
     <joint name="left_wheel_joint" type="continuous">
         <parent link="base_link"/>
         <child link="left_wheel"/>
-        <origin xyz="0 0.175 0" rpy="-${pi/2} 0 0"/>
+        <origin xyz="0 0.0905 0" rpy="-${pi/2} 0 0"/>
         <axis xyz="0 0 1"/>
     </joint>
@@ -69,5 +136,5 @@
             <origin xyz="0 0 0" rpy="0 0 0"/>
             <geometry>
-                <cylinder radius="0.0325" length="0.026"/>
+                <cylinder radius="0.0345" length="0.026"/>
             </geometry>
             <material name="dark_grey"/>
@@ -76,16 +143,16 @@
             <origin xyz="0 0 0" rpy="0 0 0"/>
             <geometry>
-                <sphere radius="0.0325"/>
-            </geometry>
-        </collision>
-        <xacro:inertial_cylinder mass="0.1" length="0.026" radius="0.0325">
+                <sphere radius="0.0345"/>
+            </geometry>
+        </collision>
+        <xacro:inertial_cylinder mass="0.1" length="0.026" radius="0.0345">
             <origin xyz="0 0 0" rpy="0 0 0"/>
         </xacro:inertial_cylinder>
     </link>
-    <!-- RIGHT WHEEL LINK -->
+    <!-- ==================== RIGHT WHEEL ==================== -->
     <joint name="right_wheel_joint" type="continuous">
         <parent link="base_link"/>
         <child link="right_wheel"/>
-        <origin xyz="0 -0.175 0" rpy="${pi/2} 0 0"/>
+        <origin xyz="0 -0.0905 0" rpy="${pi/2} 0 0"/>
         <axis xyz="0 0 -1"/>
     </joint>
@@ -94,5 +161,5 @@
             <origin xyz="0 0 0" rpy="0 0 0"/>
             <geometry>
-                <cylinder radius="0.0325" length="0.026"/>
+                <cylinder radius="0.0345" length="0.026"/>
             </geometry>
             <material name="dark_grey"/>
@@ -101,21 +168,26 @@
             <origin xyz="0 0 0" rpy="0 0 0"/>
             <geometry>
-                <sphere radius="0.0325"/>
-            </geometry>
-        </collision>
-        <xacro:inertial_cylinder mass="0.1" length="0.026" radius="0.0325">
+                <sphere radius="0.0345"/>
+            </geometry>
+        </collision>
+        <xacro:inertial_cylinder mass="0.1" length="0.026" radius="0.0345">
             <origin xyz="0 0 0" rpy="0 0 0"/>
         </xacro:inertial_cylinder>
     </link>
-    <!--caster wheel link -->
+    <!-- ==================== CASTER WHEEL ==================== -->
+    <!--
+      Passive front caster, 190 mm forward of drive axle.
+      Relative to chassis link: x = 0.190 + 0.147 = 0.337 m
+      Small sphere (radius 0.015m) at z = -0.0195 so it contacts ground
+    -->
     <joint name="caster_wheel_joint" type="fixed">
         <parent link="chassis"/>
         <child link="caster_wheel"/>
-        <origin xyz="0.24 0 0"/>
+        <origin xyz="0.337 0 -0.0195"/>
     </joint>
     <link name="caster_wheel">
         <visual>
             <geometry>
-                <sphere radius="0.0325"/>
+                <sphere radius="0.015"/>
             </geometry>
             <material name="silver"/>
@@ -123,61 +195,10 @@
         <collision>
             <geometry>
-                <sphere radius="0.0325"/>
-            </geometry>
-        </collision>
-        <xacro:inertial_sphere mass="0.1" radius="0.0325">
+                <sphere radius="0.015"/>
+            </geometry>
+        </collision>
+        <xacro:inertial_sphere mass="0.05" radius="0.015">
             <origin xyz="0 0 0" rpy="0 0 0"/>
         </xacro:inertial_sphere>
     </link>
-    <!-- ==================== GAZEBO COLORS ==================== -->
-    <!-- Gazebo Harmonic uses these tags to apply colors in simulation -->
-    <!-- Chassis: Orange -->
-    <gazebo reference="chassis">
-        <material>
-            <ambient>1.0 0.3 0.0 1</ambient>
-            <diffuse>1.0 0.3 0.0 1</diffuse>
-            <specular>0.6 0.6 0.6 1</specular>
-        </material>
-    </gazebo>
-    <!-- Wheels: Dark Grey with high friction for traction -->
-    <gazebo reference="left_wheel">
-        <mu1>100</mu1>
-        <mu2>50</mu2>
-        <kp>1000000.0</kp>
-        <kd>1.0</kd>
-        <minDepth>0.001</minDepth>
-        <maxVel>0.0</maxVel>
-        <material>
-            <ambient>0.2 0.2 0.2 1</ambient>
-            <diffuse>0.2 0.2 0.2 1</diffuse>
-            <specular>0.3 0.3 0.3 1</specular>
-        </material>
-    </gazebo>
-    <gazebo reference="right_wheel">
-        <mu1>100</mu1>
-        <mu2>50</mu2>
-        <kp>1000000.0</kp>
-        <kd>1.0</kd>
-        <minDepth>0.001</minDepth>
-        <maxVel>0.0</maxVel>
-        <material>
-            <ambient>0.2 0.2 0.2 1</ambient>
-            <diffuse>0.2 0.2 0.2 1</diffuse>
-            <specular>0.3 0.3 0.3 1</specular>
-        </material>
-    </gazebo>
-    <!-- Caster: Silver with near-zero friction for free pivot -->
-    <gazebo reference="caster_wheel">
-        <mu1>0.001</mu1>
-        <mu2>0.001</mu2>
-        <kp>1000000.0</kp>
-        <kd>1.0</kd>
-        <minDepth>0.001</minDepth>
-        <maxVel>0.0</maxVel>
-        <material>
-            <ambient>0.75 0.75 0.75 1</ambient>
-            <diffuse>0.75 0.75 0.75 1</diffuse>
-            <specular>0.8 0.8 0.8 1</specular>
-        </material>
-    </gazebo>
 </robot>

Commit message: feat: back-port validated improvements from simulation branch
Selectively applied improvements from feature/lattepanda-alpha-daniel-sim
that were validated through Gazebo simulation testing. No Gazebo dependencies
introduced — hardware branch remains clean.

URDF visual improvements (robot_core.xacro):
  - Added motor housing cylinders (r=14mm, l=40mm) at chassis (0.147, ±0.065)
  - Added caster mount bracket (20×15×40mm) at chassis (0.337, 0, 0.015)
  - Added LiDAR riser post (40×40×25mm) at chassis (0.04, 0, 0.0675)

LiDAR position fix (lidar_hardware.xacro):
  - Moved laser_frame from x=0.106 to x=0.04 (rear edge placement)
  - Matches measured physical placement on Daniel's robot

Nav2 Jazzy pipeline fix (nav2_params_hardware.yaml):
  - Added collision_monitor config (cmd_vel_smoothed → cmd_vel relay)
  - Added docking_server config (required by Jazzy lifecycle_manager)
  - Added route_server config (required by Jazzy lifecycle_manager)

Navigation launch fix (navigation_hardware.launch.py):
  - Added velocity_smoother node (cmd_vel_nav → cmd_vel_smoothed)
  - Added collision_monitor node (cmd_vel_smoothed → cmd_vel)
  - Fixed controller_server remapping: cmd_vel → cmd_vel_nav
  - Updated lifecycle_manager node_names list

RViz view improvement (nav2_view.rviz):
  - Changed from Orbit to TopDownOrtho for better 2D navigation view

Package dependency (package.xml):
  - Added nav2_lifecycle_manager exec_depend

File: description/lidar_hardware.xacro (robot description, xacro)
@@ -4,8 +4,8 @@
     RPLidar C1 — Real Hardware Link/Joint
     Physical placement on Daniel's robot:
-      - 106 mm from rear edge of chassis (toward front)
+      - Near the rear edge of the chassis (x=0.04 in chassis frame)
       - Centered laterally (y = 0)
-      - Mounted on top of chassis, ~0.10m above base_link
-      - Relative to chassis link origin (at rear edge): x=0.106, y=0, z=0.10
+      - Mounted on a wooden riser above the chassis, ~0.10m above base_link
+      - Relative to chassis link origin (at rear edge): x=0.04, y=0, z=0.10
     The real RPLidar C1 publishes /scan via rplidar_ros driver node.
     No Gazebo sensor plugin needed.
@@ -14,5 +14,5 @@
     <parent link="chassis"/>
     <child link="laser_frame"/>
-    <origin xyz="0.106 0 0.10" rpy="0 0 0"/>
+    <origin xyz="0.04 0 0.10" rpy="0 0 0"/>
   </joint>
   <link name="laser_frame">

File: description/robot_core.xacro (robot description, xacro)
@@ -18,5 +18,5 @@
       Drive axle: 147 mm from rear edge
       Caster:     190 mm forward of drive axle
-      LiDAR:      106 mm from rear edge, centered laterally
+      LiDAR:      Near rear edge (x=0.04 in chassis frame), centered laterally
       Coordinate convention:
         base_link at drive axle center, X-forward, Z-up
@@ -120,4 +120,41 @@
         </visual>
     </link>
+    <!-- ==================== MOTOR HOUSINGS ==================== -->
+    <!--
+      DC motor cylinders between support posts and wheels.
+      Oriented along Y axis (perpendicular to chassis).
+      Radius ~14mm, length ~40mm — bridges from support post to wheel.
+      Centered at wheel X position, between post and wheel in Y.
+    -->
+    <!-- Left motor -->
+    <joint name="left_motor_joint" type="fixed">
+        <parent link="chassis"/>
+        <child link="left_motor"/>
+        <origin xyz="0.147 0.065 0" rpy="0 0 0"/>
+    </joint>
+    <link name="left_motor">
+        <visual>
+            <origin xyz="0 0 0" rpy="${pi/2} 0 0"/>
+            <geometry>
+                <cylinder radius="0.014" length="0.040"/>
+            </geometry>
+            <material name="dark_grey"/>
+        </visual>
+    </link>
+    <!-- Right motor -->
+    <joint name="right_motor_joint" type="fixed">
+        <parent link="chassis"/>
+        <child link="right_motor"/>
+        <origin xyz="0.147 -0.065 0" rpy="0 0 0"/>
+    </joint>
+    <link name="right_motor">
+        <visual>
+            <origin xyz="0 0 0" rpy="${pi/2} 0 0"/>
+            <geometry>
+                <cylinder radius="0.014" length="0.040"/>
+            </geometry>
+            <material name="dark_grey"/>
+        </visual>
+    </link>
     <!-- ==================== LEFT WHEEL ==================== -->
     <!--
@@ -175,4 +212,24 @@
         </xacro:inertial_cylinder>
     </link>
+    <!-- ==================== CASTER MOUNT BRACKET ==================== -->
+    <!--
+      Vertical bracket connecting chassis bottom (z=0.035) to caster area.
+      Fills the visual gap between the chassis plate and the caster ball.
+      Height: 40mm, from z=-0.005 to z=0.035 (chassis bottom).
+    -->
+    <joint name="caster_mount_joint" type="fixed">
+        <parent link="chassis"/>
+        <child link="caster_mount"/>
+        <origin xyz="0.337 0 0.015" rpy="0 0 0"/>
+    </joint>
+    <link name="caster_mount">
+        <visual>
+            <origin xyz="0 0 0" rpy="0 0 0"/>
+            <geometry>
+                <box size="0.020 0.015 0.040"/>
+            </geometry>
+            <material name="silver"/>
+        </visual>
+    </link>
     <!-- ==================== CASTER WHEEL ==================== -->
     <!--
@@ -202,3 +259,24 @@
         </xacro:inertial_sphere>
     </link>
+    <!-- ==================== LIDAR RISER POST ==================== -->
+    <!--
+      Wooden post supporting the LiDAR above the chassis.
+      Fills the gap between chassis top (z=0.055) and LiDAR bottom (z=0.08).
+      Height: 25mm, centered at z=0.0675.
+      Placed near the rear edge of the chassis (x=0.04 in chassis frame).
+    -->
+    <joint name="lidar_riser_joint" type="fixed">
+        <parent link="chassis"/>
+        <child link="lidar_riser"/>
+        <origin xyz="0.04 0 0.0675" rpy="0 0 0"/>
+    </joint>
+    <link name="lidar_riser">
+        <visual>
+            <origin xyz="0 0 0" rpy="0 0 0"/>
+            <geometry>
+                <box size="0.040 0.040 0.025"/>
+            </geometry>
+            <material name="wood"/>
+        </visual>
+    </link>
 </robot>

Commit message: updated the lidar position

File: description/lidar_hardware.xacro (robot description, xacro)
@@ -4,8 +4,8 @@
     RPLidar C1 — Real Hardware Link/Joint
     Physical placement on Daniel's robot:
-      - Near the rear edge of the chassis (x=0.04 in chassis frame)
+      - At the front edge of the chassis, above the caster wheel (x=0.337 in chassis frame)
       - Centered laterally (y = 0)
       - Mounted on a wooden riser above the chassis, ~0.10m above base_link
-      - Relative to chassis link origin (at rear edge): x=0.04, y=0, z=0.10
+      - Relative to chassis link origin (at rear edge): x=0.337, y=0, z=0.10
     The real RPLidar C1 publishes /scan via rplidar_ros driver node.
     No Gazebo sensor plugin needed.
@@ -14,5 +14,5 @@
     <parent link="chassis"/>
     <child link="laser_frame"/>
-    <origin xyz="0.04 0 0.10" rpy="0 0 0"/>
+    <origin xyz="0.337 0 0.10" rpy="0 0 0"/>
   </joint>
   <link name="laser_frame">

File: description/robot_core.xacro (robot description, xacro)
@@ -264,10 +264,10 @@
       Fills the gap between chassis top (z=0.055) and LiDAR bottom (z=0.08).
       Height: 25mm, centered at z=0.0675.
-      Placed near the rear edge of the chassis (x=0.04 in chassis frame).
+      Placed at the front edge of the chassis, above the caster wheel (x=0.337 in chassis frame).
     -->
     <joint name="lidar_riser_joint" type="fixed">
         <parent link="chassis"/>
         <child link="lidar_riser"/>
-        <origin xyz="0.04 0 0.0675" rpy="0 0 0"/>
+        <origin xyz="0.337 0 0.0675" rpy="0 0 0"/>
     </joint>
     <link name="lidar_riser">

Commit message: "Fixed autonomous navigation script "

File: description/lidar_hardware.xacro (robot description, xacro)
@@ -4,15 +4,15 @@
     RPLidar C1 — Real Hardware Link/Joint
     Physical placement on Daniel's robot:
-      - At the front edge of the chassis, above the caster wheel (x=0.337 in chassis frame)
+      - At the front of the chassis, above the caster wheel
       - Centered laterally (y = 0)
       - Mounted on a wooden riser above the chassis, ~0.10m above base_link
-      - Relative to chassis link origin (at rear edge): x=0.337, y=0, z=0.10
-    The real RPLidar C1 publishes /scan via rplidar_ros driver node.
-    No Gazebo sensor plugin needed.
+      - Yaw rotated 180° (π rad) because the RPLidar C1 connector faces backward
+        on the robot, so its internal 0° points rearward — the yaw flips it to
+        align with the robot's +X forward direction.
   -->
   <joint name="laser_joint" type="fixed">
     <parent link="chassis"/>
     <child link="laser_frame"/>
-    <origin xyz="0.337 0 0.10" rpy="0 0 0"/>
+    <origin xyz="0.36 0 0.10" rpy="0 0 ${pi}"/>
   </joint>
   <link name="laser_frame">

File: description/robot_core.xacro (robot description, xacro)
@@ -17,6 +17,6 @@
         Center-to-center:      181 mm  (0.181 m)
       Drive axle: 147 mm from rear edge
-      Caster:     190 mm forward of drive axle
-      LiDAR:      Near rear edge (x=0.04 in chassis frame), centered laterally
+      Caster:     190 mm forward of drive axle (front of robot)
+      LiDAR:      At the front, above the caster (x≈0.36 in chassis frame), yaw rotated 180°
       Coordinate convention:
         base_link at drive axle center, X-forward, Z-up
